File: PCB/Tutorial.kicad_pcb (KiCad board)
At the start: 2 copper layers, 100 x 100 mm, 50 parts, among them J2 Conn_01x02, J3 Conn_01x05, J4 UJ20-C-H-G-SMT-2A-P16-TR, Q1 MMBT2222A, Q2 MMBT2222A, Q3 AO3401A, Q4 NPN, SW1 SW_Push, SW2 SW_Push, U1 NCP1117-3.3_SOT223, U2 ESP32-WROOM-32, U3 CH340C, U4 SHT30-DIS

Commit message: Fixed pcb
Parts:
- removed R9: 2k, Resistor_SMD:R_0805_2012Metric
- C2: value 10uF -> 100nF
Connections:
- R10 pad 1: IO34 -> Net-(J3-Pin_2)
- R10 pad 2: GND -> IO34
Changed lines of the file:
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@@
 			)
 		)
+		(property "Sim.Device" "SW"
+			(at 0 0 0)
+			(unlocked yes)
+			(layer "F.Fab")
+			(hide yes)
+			(effects
+				(font
+					(size 1 1)
+					(thickness 0.15)
+				)
+			)
+		)
+		(property "Sim.Type" "V"
+			(at 0 0 0)
+			(unlocked yes)
+			(layer "F.Fab")
+			(hide yes)
+			(effects
+				(font
+					(size 1 1)
+					(thickness 0.15)
+				)
+			)
+		)
+		(property "Sim.Pins" "1=ctrl+ 2=ctrl-"
+			(at 0 0 0)
+			(unlocked yes)
+			(layer "F.Fab")
+			(hide yes)
+			(effects
+				(font
+					(size 1 1)
+					(thickness 0.15)
+				)
+			)
+		)
 		(sheetname "/")
 		(sheetfile "Tutorial.kicad_sch")
@@
 			)
 		)
-		(property "Value" "10uF"
+		(property "Value" "100nF"
 			(at 0 1.68 0)
 			(layer "F.Fab")
@@
 			(layers "F.Cu" "F.Mask" "F.Paste")
 			(roundrect_rratio 0.243902)
-			(net "IO34")
+			(net "Net-(J3-Pin_2)")
 			(pintype "passive")
 		)
@@
 			(layers "F.Cu" "F.Mask" "F.Paste")
 			(roundrect_rratio 0.243902)
-			(net "GND")
+			(net "IO34")
 			(pintype "passive")
 		)
@@
 			)
 		)
+		(property "Sim.Device" "D"
+			(at 0 0 180)
+			(unlocked yes)
+			(layer "F.Fab")
+			(hide yes)
+			(effects
+				(font
+					(size 1 1)
+					(thickness 0.15)
+				)
+			)
+		)
+		(property "Sim.Pins" "1=A 2=K"
+			(at 0 0 180)
+			(unlocked yes)
+			(layer "F.Fab")
+			(hide yes)
+			(effects
+				(font
+					(size 1 1)
+					(thickness 0.15)
+				)
+			)
+		)
 		(property ki_fp_filters "TO-???* *_Diode_* *SingleDiode* D_*")
 		(sheetname "/")
@@
 		)
 	)
-	(footprint "Resistor_SMD:R_0805_2012Metric"
-		(layer "F.Cu")
-		(at 56.7125 86.26)
-		(descr "Resistor SMD 0805 (2012 Metric), square (rectangular) end terminal, IPC-7351 nominal, (Body size source: IPC-SM-782 page 72, https://www.pcb-3d.com/wordpress/wp-content/uploads/ipc-sm-782a_amendment_1_and_2.pdf)")
-		(tags "resistor")
-		(property "Reference" "R9"
-			(at 0 -1.65 0)
-			(layer "F.SilkS")
-			(effects
-				(font
-					(size 1 1)
-					(thickness 0.15)
-				)
-			)
-		)
-		(property "Value" "2k"
-			(at 0 1.65 0)
-			(layer "F.Fab")
-			(effects
-				(font
-					(size 1 1)
-					(thickness 0.15)
-				)
-			)
-		)
-		(property "Datasheet" ""
-			(at 0 0 0)
-			(layer "F.Fab")
-			(hide yes)
-			(effects
-				(font
-					(size 1.27 1.27)
-				)
-			)
-		)
-		(property "Description" "Resistor"
-			(at 0 0 0)
-			(layer "F.Fab")
-			(hide yes)
-			(effects
-				(font
-					(size 1.27 1.27)
-				)
-			)
-		)
-		(property ki_fp_filters "R_*")
-		(sheetname "/")
-		(sheetfile "Tutorial.kicad_sch")
-		(units
-			(unit
-				(name "A")
-				(pins "1" "2")
-			)
-		)
-		(attr smd)
-		(duplicate_pad_numbers_are_jumpers no)
-		(fp_line
-			(start -0.227064 -0.735)
-			(end 0.227064 -0.735)
-			(stroke
-				(width 0.12)
-				(type solid)
-			)
-			(layer "F.SilkS")
-		)
-		(fp_line
-			(start -0.227064 0.735)
-			(end 0.227064 0.735)
-			(stroke
-				(width 0.12)
-				(type solid)
-			)
-			(layer "F.SilkS")
-		)
-		(fp_rect
-			(start -1.68 -0.95)
-			(end 1.68 0.95)
-			(stroke
-				(width 0.05)
-				(type solid)
-			)
-			(fill no)
-			(layer "F.CrtYd")
-		)
-		(fp_rect
-			(start -1 -0.625)
-			(end 1 0.625)
-			(stroke
-				(width 0.1)
-				(type solid)
-			)
-			(fill no)
-			(layer "F.Fab")
-		)
-		(fp_text user "${REFERENCE}"
-			(at 0 0 0)
-			(layer "F.Fab")
-			(effects
-				(font
-					(size 0.5 0.5)
-					(thickness 0.08)
-				)
-			)
-		)
-		(pad "1" smd roundrect
-			(at -0.9125 0)
-			(size 1.025 1.4)
-			(layers "F.Cu" "F.Mask" "F.Paste")
-			(roundrect_rratio 0.243902)
-			(net "Net-(J3-Pin_2)")
-			(pintype "passive")
-		)
-		(pad "2" smd roundrect
-			(at 0.9125 0)
-			(size 1.025 1.4)
-			(layers "F.Cu" "F.Mask" "F.Paste")
-			(roundrect_rratio 0.243902)
-			(net "IO34")
-			(pintype "passive")
-		)
-		(embedded_fonts no)
-		(model "${KICAD10_3DMODEL_DIR}/Resistor_SMD.3dshapes/R_0805_2012Metric.step"
-			(offset
-				(xyz 0 0 0)
-			)
-			(scale
-				(xyz 1 1 1)
-			)
-			(rotate
-				(xyz 0 0 0)
-			)
-		)
-	)
 	(footprint "RF_Module:ESP32-WROOM-32"
 		(layer "F.Cu")
@@
 			)
 		)
+		(property "Sim.Device" "PMOS"
+			(at 0 0 180)
+			(unlocked yes)
+			(layer "F.Fab")
+			(hide yes)
+			(effects
+				(font
+					(size 1 1)
+					(thickness 0.15)
+				)
+			)
+		)
+		(property "Sim.Type" "VDMOS"
+			(at 0 0 180)
+			(unlocked yes)
+			(layer "F.Fab")
+			(hide yes)
+			(effects
+				(font
+					(size 1 1)
+					(thickness 0.15)
+				)
+			)
+		)
+		(property "Sim.Pins" "1=D 2=G 3=S"
+			(at 0 0 180)
+			(unlocked yes)
+			(layer "F.Fab")
+			(hide yes)
+			(effects
+				(font
+					(size 1 1)
+					(thickness 0.15)
+				)
+			)
+		)
 		(property ki_fp_filters "SOT?23*")
 		(sheetname "/")
@@
 			)
 		)
+		(property "Sim.Device" "D"
+			(at 0 0 180)
+			(unlocked yes)
+			(layer "F.Fab")
+			(hide yes)
+			(effects
+				(font
+					(size 1 1)
+					(thickness 0.15)
+				)
+			)
+		)
+		(property "Sim.Pins" "1=A 2=K"
+			(at 0 0 180)
+			(unlocked yes)
+			(layer "F.Fab")
+			(hide yes)
+			(effects
+				(font
+					(size 1 1)
+					(thickness 0.15)
+				)
+			)
+		)
 		(property ki_fp_filters "TO-???* *_Diode_* *SingleDiode* D_*")
 		(sheetname "/")
@@
 	)
 	(segment
-		(start 55.74 86.32)
-		(end 55.8 86.26)
-		(width 0.2)
-		(layer "F.Cu")
-		(net "Net-(J3-Pin_2)")
-	)
-	(segment
-		(start 52.6 86.32)
-		(end 55.74 86.32)
-		(width 0.2)
-		(layer "F.Cu")
-		(net "Net-(J3-Pin_2)")
-	)
-	(segment
-		(start 58.4 91.06)
-		(end 54.8 91.06)
-		(width 0.2)
-		(layer "F.Cu")
-		(net "Net-(J3-Pin_3)")
-	)
-	(segment
-		(start 54.8 91.06)
-		(end 52.6 88.86)
-		(width 0.2)
-		(layer "F.Cu")
-		(net "Net-(J3-Pin_3)")
-	)
-	(segment
-		(start 64.35 92.01)
-		(end 64.4 92.06)
-		(width 0.2)
-		(layer "F.Cu")
-		(net "Net-(Q3-G)")
-	)
-	(segment
-		(start 60.275 92.01)
-		(end 64.35 92.01)
-		(width 0.2)
-		(layer "F.Cu")
-		(net "Net-(Q3-G)")
-	)
-	(segment
-		(start 43.0484 92.7933)
-		(end 36.9933 92.7933)
-		(width 0.2)
-		(layer "F.Cu")
-		(net "Net-(D1-A)")
-	)
-	(segment
-		(start 36.9933 92.7933)
-		(end 24.8 80.6)
-		(width 0.2)
-		(layer "F.Cu")
-		(net "Net-(D1-A)")
-	)
-	(segment
 		(start 55.2028 85.0542)
 		(end 56.4192 85.0542)
@@
 	)
 	(segment
+		(start 55.74 86.32)
+		(end 55.8 86.26)
+		(width 0.2)
+		(layer "F.Cu")
+		(net "Net-(J3-Pin_2)")
+	)
+	(segment
+		(start 52.6 86.32)
+		(end 55.74 86.32)
+		(width 0.2)
+		(layer "F.Cu")
+		(net "Net-(J3-Pin_2)")
+	)
+	(segment
+		(start 58.4 91.06)
+		(end 54.8 91.06)
+		(width 0.2)
+		(layer "F.Cu")
+		(net "Net-(J3-Pin_3)")
+	)
+	(segment
+		(start 54.8 91.06)
+		(end 52.6 88.86)
+		(width 0.2)
+		(layer "F.Cu")
+		(net "Net-(J3-Pin_3)")
+	)
+	(segment
+		(start 64.35 92.01)
+		(end 64.4 92.06)
+		(width 0.2)
+		(layer "F.Cu")
+		(net "Net-(Q3-G)")
+	)
+	(segment
+		(start 60.275 92.01)
+		(end 64.35 92.01)
+		(width 0.2)
+		(layer "F.Cu")
+		(net "Net-(Q3-G)")
+	)
+	(segment
+		(start 43.0484 92.7933)
+		(end 36.9933 92.7933)
+		(width 0.2)
+		(layer "F.Cu")
+		(net "Net-(D1-A)")
+	)
+	(segment
+		(start 36.9933 92.7933)
+		(end 24.8 80.6)
+		(width 0.2)
+		(layer "F.Cu")
+		(net "Net-(D1-A)")
+	)
+	(segment
