File: PCB/Tutorial.kicad_sch (KiCad schematic)
At the start: 50 parts, among them J2 Conn_01x02, J3 Conn_01x05, J4 UJ20-C-H-G-SMT-2A-P16-TR, Q1 MMBT2222A, Q2 MMBT2222A, Q3 AO3401A, Q4 NPN, SW1 SW_Push, SW2 SW_Push, U1 NCP1117-3.3_SOT223, U2 ESP32-WROOM-32, U3 CH340C, U4 SHT30-DIS

Commit message: Fixed pcb
Parts:
- removed R9: 2k, Resistor_SMD:R_0805_2012Metric, symbol Device:R
- C2: value 10uF -> 100nF
Connections:
- net GND: no longer R10.2
- net IO34: now also R10.2; no longer R10.1
- net at J3.2 (Pin_2): now also R10.1
Other:
- moved on the sheet: R10
Changed lines of the file:
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@@
 	)
 	(junction
-		(at 26.67 151.13)
-		(diameter 0)
-		(color 0 0 0 0)
-	)
-	(junction
 		(at 90.17 144.78)
 		(diameter 0)
@@
 	(wire
 		(pts
-			(xy 26.67 143.51) (xy 26.67 142.24)
-		)
-		(stroke
-			(width 0)
-			(type default)
-		)
-	)
-	(wire
-		(pts
 			(xy 38.1 48.26) (xy 40.64 48.26)
 		)
@@
 	(wire
 		(pts
-			(xy 21.59 151.13) (xy 26.67 151.13)
+			(xy 26.67 143.51) (xy 26.67 142.24)
 		)
 		(stroke
@@
 	(global_label "IO34"
 		(shape input)
-		(at 21.59 151.13 180)
+		(at 26.67 151.13 270)
 		(fields_autoplaced yes)
 		(effects
@@
 		)
 		(property "Intersheetrefs" "${INTERSHEET_REFS}"
-			(at 14.2505 151.13 0)
+			(at 26.67 158.4695 90)
 			(hide yes)
 			(show_name no)
@@
 	)
 	(symbol
-		(lib_id "power:GND")
-		(at 26.67 158.75 0)
-		(unit 1)
-		(body_style 1)
-		(exclude_from_sim no)
-		(in_bom yes)
-		(on_board yes)
-		(in_pos_files yes)
-		(dnp no)
-		(fields_autoplaced yes)
-		(property "Reference" "#PWR014"
-			(at 26.67 165.1 0)
-			(hide yes)
-			(show_name no)
-			(do_not_autoplace no)
-			(effects
-				(font
-					(size 1.27 1.27)
-				)
-			)
-		)
-		(property "Value" "GND"
-			(at 26.67 163.83 0)
-			(show_name no)
-			(do_not_autoplace no)
-			(effects
-				(font
-					(size 1.27 1.27)
-				)
-			)
-		)
-		(property "Footprint" ""
-			(at 26.67 158.75 0)
-			(hide yes)
-			(show_name no)
-			(do_not_autoplace no)
-			(effects
-				(font
-					(size 1.27 1.27)
-				)
-			)
-		)
-		(property "Datasheet" ""
-			(at 26.67 158.75 0)
-			(hide yes)
-			(show_name no)
-			(do_not_autoplace no)
-			(effects
-				(font
-					(size 1.27 1.27)
-				)
-			)
-		)
-		(property "Description" "Power symbol creates a global label with name \"GND\" , ground"
-			(at 26.67 158.75 0)
-			(hide yes)
-			(show_name no)
-			(do_not_autoplace no)
-			(effects
-				(font
-					(size 1.27 1.27)
-				)
-			)
-		)
-		(pin "1"
-		)
-		(instances
-			(project "Tutorial"
-				(path "/8c660991-c4f8-4c22-b15c-53b2a9e6fa68"
-					(reference "#PWR014")
-					(unit 1)
-				)
-			)
-		)
-	)
-	(symbol
 		(lib_id "Device:C")
 		(at 176.53 128.27 90)
@@
 	(symbol
 		(lib_id "Device:R")
-		(at 26.67 154.94 0)
+		(at 26.67 147.32 0)
 		(unit 1)
 		(body_style 1)
@@
 		(fields_autoplaced yes)
 		(property "Reference" "R10"
-			(at 29.21 153.6699 0)
+			(at 29.21 146.0499 0)
 			(show_name no)
 			(do_not_autoplace no)
@@
 		)
 		(property "Value" "1k"
-			(at 29.21 156.2099 0)
+			(at 29.21 148.5899 0)
 			(show_name no)
 			(do_not_autoplace no)
@@
 		)
 		(property "Footprint" "Resistor_SMD:R_0805_2012Metric"
-			(at 24.892 154.94 90)
+			(at 24.892 147.32 90)
 			(hide yes)
 			(show_name no)
@@
 		)
 		(property "Datasheet" ""
-			(at 26.67 154.94 0)
+			(at 26.67 147.32 0)
 			(hide yes)
 			(show_name no)
@@
 		)
 		(property "Description" "Resistor"
-			(at 26.67 154.94 0)
+			(at 26.67 147.32 0)
 			(hide yes)
 			(show_name no)
@@
 			)
 		)
-		(property "Value" "10uF"
+		(property "Value" "100nF"
 			(at 115.57 78.7399 0)
 			(show_name no)
@@
 					(unit 1)
 				)
-			)
-		)
-	)
-	(symbol
-		(lib_id "Device:R")
-		(at 26.67 147.32 0)
-		(unit 1)
-		(body_style 1)
-		(exclude_from_sim no)
-		(in_bom yes)
-		(on_board yes)
-		(in_pos_files yes)
-		(dnp no)
-		(property "Reference" "R9"
-			(at 21.844 147.32 0)
-			(show_name no)
-			(do_not_autoplace no)
-			(effects
-				(font
-					(size 1.27 1.27)
-				)
-				(justify left)
-			)
-		)
-		(property "Value" "2k"
-			(at 21.844 149.86 0)
-			(show_name no)
-			(do_not_autoplace no)
-			(effects
-				(font
-					(size 1.27 1.27)
-				)
-				(justify left)
-			)
-		)
-		(property "Footprint" "Resistor_SMD:R_0805_2012Metric"
-			(at 24.892 147.32 90)
-			(hide yes)
-			(show_name no)
-			(do_not_autoplace no)
-			(effects
-				(font
-					(size 1.27 1.27)
-				)
-			)
-		)
-		(property "Datasheet" ""
-			(at 26.67 147.32 0)
-			(hide yes)
-			(show_name no)
-			(do_not_autoplace no)
-			(effects
-				(font
-					(size 1.27 1.27)
-				)
-			)
-		)
-		(property "Description" "Resistor"
-			(at 26.67 147.32 0)
-			(hide yes)
-			(show_name no)
-			(do_not_autoplace no)
-			(effects
-				(font
-					(size 1.27 1.27)
-				)
-			)
-		)
-		(pin "2"
-		)
-		(pin "1"
-		)
-		(instances
-			(project "Tutorial"
-				(path "/8c660991-c4f8-4c22-b15c-53b2a9e6fa68"
-					(reference "R9")
-					(unit 1)
-				)
